Commit message: updating my_bot config files for skid driving

File: urdf/my_bot.xacro (robot description, xacro)
@@ -11,10 +11,10 @@
     <pose>0 0 0.5 0 0 0</pose>
     <inertial>
-      <mass value="5.0"/>
+      <mass value="10.0"/>
       <origin xyz="0.0 0 0" rpy=" 0 0 0"/>
       <inertia
-          ixx="0.1" ixy="0" ixz="0"
-          iyy="0.1" iyz="0"
-          izz="0.1"
+          ixx="1.0" ixy="0" ixz="0"
+          iyy="1.0" iyz="0"
+          izz="1.0"
       />
     </inertial>
@@ -22,5 +22,5 @@
       <origin xyz="0 0 0" rpy=" 0 0 0"/>
       <geometry>
-        <box size=".8 .2 .02"/>
+        <box size=".22 .2 .1"/>
       </geometry>
     </collision>
@@ -28,5 +28,5 @@
       <origin xyz="0 0 0" rpy=" 0 0 0"/>
       <geometry>
-        <box size=".8 .2 .02"/>
+        <box size=".22 .2 .1"/>
       </geometry>
     </visual>
@@ -51,8 +51,8 @@
         <friction>
           <ode>
-            <mu>0</mu>
-            <mu2>0</mu2>
-            <slip1>1.0</slip1>
-            <slip2>1.0</slip2>
+            <mu>0.0</mu>
+            <mu2>0.0</mu2>
+	    <slip1>1.0</slip1>
+	    <slip2>1.0</slip2>
           </ode>
         </friction>
@@ -67,5 +67,5 @@
   </link>
   <joint type="continuous" name="front_right_wheel_hinge">
-    <origin xyz="0.3 -0.15 0" rpy="0 0 0"/>
+    <origin xyz="0.11 -0.15 0" rpy="0 0 0"/>
     <child link="front_right_wheel"/>
     <parent link="chassis"/>
@@ -93,8 +93,8 @@
         <friction>
           <ode>
-            <mu>0</mu>
-            <mu2>0</mu2>
-            <slip1>1.0</slip1>
-            <slip2>1.0</slip2>
+            <mu>0.0</mu>
+            <mu2>0.0</mu2>
+	    <slip1>1.0</slip1>
+	    <slip2>1.0</slip2>
           </ode>
         </friction>
@@ -109,5 +109,5 @@
   </link>
   <joint type="continuous" name="front_left_wheel_hinge">
-    <origin xyz="0.3 0.15 0" rpy="0 0 0"/>
+    <origin xyz="0.11 0.15 0" rpy="0 0 0"/>
     <child link="front_left_wheel"/>
     <parent link="chassis"/>
@@ -135,8 +135,8 @@
         <friction>
           <ode>
-            <mu>0</mu>
-            <mu2>0</mu2>
-            <slip1>1.0</slip1>
-            <slip2>1.0</slip2>
+            <mu>0.0</mu>
+            <mu2>0.0</mu2>
+	    <slip1>1.0</slip1>
+	    <slip2>1.0</slip2>
           </ode>
         </friction>
@@ -151,5 +151,5 @@
   </link>
   <joint type="continuous" name="back_right_wheel_hinge">
-    <origin xyz="-0.3 -0.15 0" rpy="0 0 0"/>
+    <origin xyz="-0.11 -0.15 0" rpy="0 0 0"/>
     <child link="back_right_wheel"/>
     <parent link="chassis"/>
@@ -177,8 +177,8 @@
         <friction>
           <ode>
-            <mu>0</mu>
-            <mu2>0</mu2>
-            <slip1>1.0</slip1>
-            <slip2>1.0</slip2>
+            <mu>0.0</mu>
+            <mu2>0.0</mu2>
+	    <slip1>1.0</slip1>
+	    <slip2>1.0</slip2>
           </ode>
         </friction>
@@ -193,5 +193,5 @@
   </link>
   <joint type="continuous" name="back_left_wheel_hinge">
-    <origin xyz="-0.3 0.15 0" rpy="0 0 0"/>
+    <origin xyz="-0.11 0.15 0" rpy="0 0 0"/>
     <child link="back_left_wheel"/>
     <parent link="chassis"/>
@@ -225,5 +225,5 @@
   </link>
   <joint type="fixed" name="camera_joint">
-    <origin xyz="0.4 0 0" rpy="0 0 0"/>
+    <origin xyz="0.11 0 0" rpy="0 0 0"/>
     <child link="camera"/>
     <parent link="chassis"/>
@@ -254,5 +254,5 @@
   </link>
   <joint type="fixed" name="hokuyo_joint">
-    <origin xyz="0.35 0 0.02" rpy="0 0 0"/>
+    <origin xyz="0.1 0 0.1" rpy="0 0 0"/>
     <child link="hokuyo"/>
     <parent link="chassis"/>

Commit message: with larger inertia they tend to follow the path and not turn around all the time

File: urdf/my_bot.xacro (robot description, xacro)
@@ -14,7 +14,7 @@
       <origin xyz="0.0 0 0" rpy=" 0 0 0"/>
       <inertia
-          ixx="1.0" ixy="0" ixz="0"
-          iyy="1.0" iyz="0"
-          izz="1.0"
+          ixx="0.5" ixy="0" ixz="0"
+          iyy="0.5" iyz="0"
+          izz="0.5"
       />
     </inertial>

File: urdf/udacity_bot.xacro (robot description, xacro)
@@ -12,9 +12,9 @@
     <inertial>
       <mass value="15.0"/>
-      <origin xyz="0.0 0 0" rpy=" 0 0 0"/>
-      <inertia
-          ixx="0.1" ixy="0" ixz="0"
-          iyy="0.1" iyz="0"
-          izz="0.1"
+      <origin xyz="0.0 0 0" rpy="0 0 0"/>
+      <inertia
+          ixx="0.3" ixy="0" ixz="0"
+          iyy="0.3" iyz="0"
+          izz="0.3"
       />
     </inertial>
